File: kicad/Pico.kicad_sch (KiCad schematic)
At the start: 14 parts, among them U1 Pico

Commit message: Rotated
Parts:
- removed R3, R6, R9: 47, Resistor_THT:R_Axial_DIN0207_L6.3mm_D2.5mm_P10.16mm_Horizontal, symbol Device:R_Small
- added RN1: 47, Resistor_THT:R_Array_SIP4, symbol Device:R_Network03_Split
- R10: renamed from R5; footprint Resistor_THT:R_Axial_DIN0207_L6.3mm_D2.5mm_P10.16mm_Horizontal -> Resistor_THT:R_Axial_DIN0204_L3.6mm_D1.6mm_P5.08mm_Horizontal
- R11: renamed from R8; footprint Resistor_THT:R_Axial_DIN0207_L6.3mm_D2.5mm_P10.16mm_Horizontal -> Resistor_THT:R_Axial_DIN0204_L3.6mm_D1.6mm_P5.08mm_Horizontal
- R4: renamed from R10; footprint Resistor_THT:R_Axial_DIN0207_L6.3mm_D2.5mm_P10.16mm_Horizontal -> Resistor_THT:R_Axial_DIN0204_L3.6mm_D1.6mm_P5.08mm_Horizontal
- R5: renamed from R11; footprint Resistor_THT:R_Axial_DIN0207_L6.3mm_D2.5mm_P10.16mm_Horizontal -> Resistor_THT:R_Axial_DIN0204_L3.6mm_D1.6mm_P5.08mm_Horizontal
- R6: renamed from R2; footprint Resistor_THT:R_Axial_DIN0207_L6.3mm_D2.5mm_P10.16mm_Horizontal -> Resistor_THT:R_Axial_DIN0204_L3.6mm_D1.6mm_P5.08mm_Horizontal
- R7: renamed from R4; footprint Resistor_THT:R_Axial_DIN0207_L6.3mm_D2.5mm_P10.16mm_Horizontal -> Resistor_THT:R_Axial_DIN0204_L3.6mm_D1.6mm_P5.08mm_Horizontal
- R8: renamed from R7; footprint Resistor_THT:R_Axial_DIN0207_L6.3mm_D2.5mm_P10.16mm_Horizontal -> Resistor_THT:R_Axial_DIN0204_L3.6mm_D1.6mm_P5.08mm_Horizontal
- R9: renamed from R1; footprint Resistor_THT:R_Axial_DIN0207_L6.3mm_D2.5mm_P10.16mm_Horizontal -> Resistor_THT:R_Axial_DIN0204_L3.6mm_D1.6mm_P5.08mm_Horizontal
- SW1: renamed from JP1; footprint Button_Switch_THT:SW_CuK_OS102011MA1QN1_SPDT_Angled -> Button_Switch_THT:SW_Slide_SPDT_Angled_CK_OS102011MA1Q
- SW2: renamed from JP2; footprint Button_Switch_THT:SW_Tactile_SPST_Angled_PTS645Vx31-2LFS -> Button_Switch_THT:SW_Tactile_SKHH_Angled
- U1: footprint pico:RPi_Pico_SMD_TH -> Pico:RaspberryPi_Pico_Common_THT_b
Connections:
- net GND: now also SW1.2 (B), SW2.1 (A), RN1.1 (R1), RN1.1 (R1), RN1.1 (R1); no longer SW1.3 (C), SW2.2 (B)
- net VGA_B: now also RN1.4 (R3.2)
- net VGA_G: now also RN1.3 (R2.2)
- net VGA_R: now also RN1.2 (R1.2)
- net at U1.30 (RUN): now also SW2.2 (B); no longer SW2.1 (A)
- net at U1.31 (GPIO26_ADC0): now also SW1.3 (C); no longer SW1.2 (B)
- net +5V: now reaches U1.39 (VSYS)
- no-connect marks 14 -> 13
Other:
- moved on the sheet: SW1, SW2
