File: kicad/connectors.kicad_sch (KiCad schematic)
At the start: 6 parts, among them J1 VGA socket, J2 CPC video port

Commit message: Rotated
Parts:
- removed J2: CPC video port, Connector_PinHeader_2.54mm:PinHeader_1x05_P2.54mm_Vertical, symbol Connector:Conn_01x05_Pin
- added J2: DE9_Pins, Connector_Dsub:DSUB-9_Pins_Horizontal_P2.77x2.54mm_EdgePinOffset9.40mm, symbol Connector:DE9_Pins
- added J3: Barrel_Jack, Connector_BarrelJack:BarrelJack_Horizontal, symbol Connector:Barrel_Jack
- added J4: Conn_01x02_Pin, Connector_JST:JST_XH_S2B-XH-A_1x02_P2.50mm_Horizontal, symbol Connector:Conn_01x02_Pin
- J1: footprint Connector_Dsub:DSUB-15-HD_Female_Horizontal_P2.29x1.98mm_EdgePinOffset3.03mm_Housed_MountingHolesOffset4.94mm -> Connector_Dsub:DSUB-15-HD_Socket_Horizontal_P2.29x2.54mm_EdgePinOffset8.35mm_Housed_MountingHolesOffset10.89mm
Connections:
- net CPC_B: now also J2.1
- net CPC_CSYNC: now also J2.7
- net CPC_G: now also J2.3
- net CPC_R: now also J2.5
- net GND: now also J2.2, J2.4, J2.6, J2.8, J2.9, J3.2, J4.2 (Pin_2)
- new net +5V: J3.1, J4.1 (Pin_1)
